File: mist.sch (KiCad schematic (older format))
At the start: 20 parts, among them SW1 SW_Push, SW10 SW_Push, SW11 SW_Push, SW12 SW_Push, SW13 SW_Push, SW14 SW_Push, SW15 SW_Push, SW16 SW_Push, SW17 SW_Push, SW18 SW_Push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

Commit message: added clickhole and gerbers
Parts:
- SW1, SW10, SW11, SW12, SW13, SW14, SW15, SW16, SW17, SW18, SW19, SW2, SW3, SW4, SW5, SW6, SW7, SW8, SW9: footprint Keebio-Parts:Kailh-PG1350-1u-NoLED -> Keebio-Parts:Kailh-PG1350-1u-Clickhole-NoLED
Changed lines of the file:
@@
 F 0 "SW1" H 4200 1185 50  0000 C CNN
 F 1 "SW_Push" H 4200 1094 50  0000 C CNN
-F 2 "Keebio-Parts:Kailh-PG1350-1u-NoLED" H 4200 1100 50  0001 C CNN
+F 2 "Keebio-Parts:Kailh-PG1350-1u-Clickhole-NoLED" H 4200 1100 50  0001 C CNN
 F 3 "~" H 4200 1100 50  0001 C CNN
 	1    4200 900
@@
 F 0 "SW5" H 6600 1185 50  0000 C CNN
 F 1 "SW_Push" H 6600 1094 50  0000 C CNN
-F 2 "Keebio-Parts:Kailh-PG1350-1u-NoLED" H 6600 1100 50  0001 C CNN
+F 2 "Keebio-Parts:Kailh-PG1350-1u-Clickhole-NoLED" H 6600 1100 50  0001 C CNN
 F 3 "~" H 6600 1100 50  0001 C CNN
 	1    6600 900
@@
 F 0 "SW4" H 6000 1185 50  0000 C CNN
 F 1 "SW_Push" H 6000 1094 50  0000 C CNN
-F 2 "Keebio-Parts:Kailh-PG1350-1u-NoLED" H 6000 1100 50  0001 C CNN
+F 2 "Keebio-Parts:Kailh-PG1350-1u-Clickhole-NoLED" H 6000 1100 50  0001 C CNN
 F 3 "~" H 6000 1100 50  0001 C CNN
 	1    6000 900
@@
 F 0 "SW3" H 5400 1185 50  0000 C CNN
 F 1 "SW_Push" H 5400 1094 50  0000 C CNN
-F 2 "Keebio-Parts:Kailh-PG1350-1u-NoLED" H 5400 1100 50  0001 C CNN
+F 2 "Keebio-Parts:Kailh-PG1350-1u-Clickhole-NoLED" H 5400 1100 50  0001 C CNN
 F 3 "~" H 5400 1100 50  0001 C CNN
 	1    5400 900
@@
 F 0 "SW2" H 4800 1185 50  0000 C CNN
 F 1 "SW_Push" H 4800 1094 50  0000 C CNN
-F 2 "Keebio-Parts:Kailh-PG1350-1u-NoLED" H 4800 1100 50  0001 C CNN
+F 2 "Keebio-Parts:Kailh-PG1350-1u-Clickhole-NoLED" H 4800 1100 50  0001 C CNN
 F 3 "~" H 4800 1100 50  0001 C CNN
 	1    4800 900
@@
 F 0 "SW6" H 4200 1935 50  0000 C CNN
 F 1 "SW_Push" H 4200 1844 50  0000 C CNN
-F 2 "Keebio-Parts:Kailh-PG1350-1u-NoLED" H 4200 1850 50  0001 C CNN
+F 2 "Keebio-Parts:Kailh-PG1350-1u-Clickhole-NoLED" H 4200 1850 50  0001 C CNN
 F 3 "~" H 4200 1850 50  0001 C CNN
 	1    4200 1650
@@
 F 0 "SW10" H 6600 1935 50  0000 C CNN
 F 1 "SW_Push" H 6600 1844 50  0000 C CNN
-F 2 "Keebio-Parts:Kailh-PG1350-1u-NoLED" H 6600 1850 50  0001 C CNN
+F 2 "Keebio-Parts:Kailh-PG1350-1u-Clickhole-NoLED" H 6600 1850 50  0001 C CNN
 F 3 "~" H 6600 1850 50  0001 C CNN
 	1    6600 1650
@@
 F 0 "SW9" H 6000 1935 50  0000 C CNN
 F 1 "SW_Push" H 6000 1844 50  0000 C CNN
-F 2 "Keebio-Parts:Kailh-PG1350-1u-NoLED" H 6000 1850 50  0001 C CNN
+F 2 "Keebio-Parts:Kailh-PG1350-1u-Clickhole-NoLED" H 6000 1850 50  0001 C CNN
 F 3 "~" H 6000 1850 50  0001 C CNN
 	1    6000 1650
@@
 F 0 "SW8" H 5400 1935 50  0000 C CNN
 F 1 "SW_Push" H 5400 1844 50  0000 C CNN
-F 2 "Keebio-Parts:Kailh-PG1350-1u-NoLED" H 5400 1850 50  0001 C CNN
+F 2 "Keebio-Parts:Kailh-PG1350-1u-Clickhole-NoLED" H 5400 1850 50  0001 C CNN
 F 3 "~" H 5400 1850 50  0001 C CNN
 	1    5400 1650
@@
 F 0 "SW7" H 4800 1935 50  0000 C CNN
 F 1 "SW_Push" H 4800 1844 50  0000 C CNN
-F 2 "Keebio-Parts:Kailh-PG1350-1u-NoLED" H 4800 1850 50  0001 C CNN
+F 2 "Keebio-Parts:Kailh-PG1350-1u-Clickhole-NoLED" H 4800 1850 50  0001 C CNN
 F 3 "~" H 4800 1850 50  0001 C CNN
 	1    4800 1650
@@
 F 0 "SW11" H 4200 2685 50  0000 C CNN
 F 1 "SW_Push" H 4200 2594 50  0000 C CNN
-F 2 "Keebio-Parts:Kailh-PG1350-1u-NoLED" H 4200 2600 50  0001 C CNN
+F 2 "Keebio-Parts:Kailh-PG1350-1u-Clickhole-NoLED" H 4200 2600 50  0001 C CNN
 F 3 "~" H 4200 2600 50  0001 C CNN
 	1    4200 2400
@@
 F 0 "SW15" H 6600 2685 50  0000 C CNN
 F 1 "SW_Push" H 6600 2594 50  0000 C CNN
-F 2 "Keebio-Parts:Kailh-PG1350-1u-NoLED" H 6600 2600 50  0001 C CNN
+F 2 "Keebio-Parts:Kailh-PG1350-1u-Clickhole-NoLED" H 6600 2600 50  0001 C CNN
 F 3 "~" H 6600 2600 50  0001 C CNN
 	1    6600 2400
@@
 F 0 "SW14" H 6000 2685 50  0000 C CNN
 F 1 "SW_Push" H 6000 2594 50  0000 C CNN
-F 2 "Keebio-Parts:Kailh-PG1350-1u-NoLED" H 6000 2600 50  0001 C CNN
+F 2 "Keebio-Parts:Kailh-PG1350-1u-Clickhole-NoLED" H 6000 2600 50  0001 C CNN
 F 3 "~" H 6000 2600 50  0001 C CNN
 	1    6000 2400
@@
 F 0 "SW13" H 5400 2685 50  0000 C CNN
 F 1 "SW_Push" H 5400 2594 50  0000 C CNN
-F 2 "Keebio-Parts:Kailh-PG1350-1u-NoLED" H 5400 2600 50  0001 C CNN
+F 2 "Keebio-Parts:Kailh-PG1350-1u-Clickhole-NoLED" H 5400 2600 50  0001 C CNN
 F 3 "~" H 5400 2600 50  0001 C CNN
 	1    5400 2400
@@
 F 0 "SW12" H 4800 2685 50  0000 C CNN
 F 1 "SW_Push" H 4800 2594 50  0000 C CNN
-F 2 "Keebio-Parts:Kailh-PG1350-1u-NoLED" H 4800 2600 50  0001 C CNN
+F 2 "Keebio-Parts:Kailh-PG1350-1u-Clickhole-NoLED" H 4800 2600 50  0001 C CNN
 F 3 "~" H 4800 2600 50  0001 C CNN
 	1    4800 2400
@@
 F 0 "SW16" H 3600 3485 50  0000 C CNN
 F 1 "SW_Push" H 3600 3394 50  0000 C CNN
-F 2 "Keebio-Parts:Kailh-PG1350-1u-NoLED" H 3600 3400 50  0001 C CNN
+F 2 "Keebio-Parts:Kailh-PG1350-1u-Clickhole-NoLED" H 3600 3400 50  0001 C CNN
 F 3 "~" H 3600 3400 50  0001 C CNN
 	1    3600 3200
@@
 F 0 "SW19" H 7200 3485 50  0000 C CNN
 F 1 "SW_Push" H 7200 3394 50  0000 C CNN
-F 2 "Keebio-Parts:Kailh-PG1350-1u-NoLED" H 7200 3400 50  0001 C CNN
+F 2 "Keebio-Parts:Kailh-PG1350-1u-Clickhole-NoLED" H 7200 3400 50  0001 C CNN
 F 3 "~" H 7200 3400 50  0001 C CNN
 	1    7200 3200
@@
 F 0 "SW18" H 6600 3485 50  0000 C CNN
 F 1 "SW_Push" H 6600 3394 50  0000 C CNN
-F 2 "Keebio-Parts:Kailh-PG1350-1u-NoLED" H 6600 3400 50  0001 C CNN
+F 2 "Keebio-Parts:Kailh-PG1350-1u-Clickhole-NoLED" H 6600 3400 50  0001 C CNN
 F 3 "~" H 6600 3400 50  0001 C CNN
 	1    6600 3200
@@
 F 0 "SW17" H 4200 3485 50  0000 C CNN
 F 1 "SW_Push" H 4200 3394 50  0000 C CNN
-F 2 "Keebio-Parts:Kailh-PG1350-1u-NoLED" H 4200 3400 50  0001 C CNN
+F 2 "Keebio-Parts:Kailh-PG1350-1u-Clickhole-NoLED" H 4200 3400 50  0001 C CNN
 F 3 "~" H 4200 3400 50  0001 C CNN
 	1    4200 3200
